Commit message: Add HDL32E support; fix LASER_3D envar names

File: urdf/accessories.urdf.xacro (robot description, xacro)
@@ -32,4 +32,5 @@
     Add/remove a 3D lidar sensor by changing the CPR_LASER_3D environment variable. The default lidar model is the Velodyne VLP16, but this can be changed with the CPR_LASER_3D_MODEL environment variable. Valid model designations are:
     - vlp16 (default)  :: Velodyne VLP16
+    - vlp32e           :: Velodyne HDL-32E
   -->
   <xacro:if value="$(optenv CPR_LASER_3D 0)">
@@ -37,7 +38,13 @@
     <xacro:if value="${lidar_3d_model == 'vlp16'}">
       <xacro:include filename="$(find velodyne_description)/urdf/VLP-16.urdf.xacro" />
-      <xacro:VLP-16 parent="$(optenv CPR_LASER_PARENT base_link)" topic="$(optenv CPR_LASER_TOPIC scan)">
-        <origin xyz="$(optenv CPR_LASER_XYZ 0 0 0)" rpy="$(optenv CPR_LASER_RPY 0 0 0)" />
+      <xacro:VLP-16 parent="$(optenv CPR_LASER_3D_PARENT base_link)" topic="$(optenv CPR_LASER_3D_TOPIC points)">
+        <origin xyz="$(optenv CPR_LASER_3D_XYZ 0 0 0)" rpy="$(optenv CPR_LASER_3D_RPY 0 0 0)" />
       </xacro:VLP-16>
+    </xacro:if>
+    <xacro:if value="${lidar_3d_model == 'hdl32e'}">
+      <xacro:include filename="$(find velodyne_description)/urdf/HDL-32E.urdf.xacro" />
+      <xacro:HDL-32E parent="$(optenv CPR_LASER_3D_PARENT base_link)" topic="$(optenv CPR_LASER_3D_TOPIC points)">
+        <origin xyz="$(optenv CPR_LASER_3D_XYZ 0 0 0)" rpy="$(optenv CPR_LASER_3D_RPY 0 0 0)" />
+      </xacro:HDL-32E>
     </xacro:if>
   </xacro:if>

Commit message: Add URDF support for Novatel SMART6 and SMART7

File: urdf/accessories.urdf.xacro (robot description, xacro)
@@ -4,5 +4,5 @@
   <material name="black"><color rgba="0.15 0.15 0.15 1.0" /></material>
   <!--
-    Add/remove a 2D lidar sensor by changing the CPR_LASER environment variable. The default lidar model is the SICK LMS1xx, but this can be changed with the CPR_LASER_MODEL environment variable. Valid model designations are:
+    Add/remove a 2D lidar sensor by changing the CPR_LASER environment variable. The default model is the SICK LMS1xx, but this can be changed with the CPR_LASER_MODEL environment variable. Valid model designations are:
     - lms1xx (default) :: SICK LMS1xx
     - ust10            :: Hokuyo UST10
@@ -13,22 +13,17 @@
       <xacro:include filename="$(find lms1xx)/urdf/sick_lms1xx.urdf.xacro" />
       <xacro:sick_lms1xx frame="$(optenv CPR_LASER_PARENT base_link)_laser" topic="$(optenv CPR_LASER_TOPIC scan)" />
-      <joint name="$(optenv CPR_LASER_PARENT base_link)_laser_joint" type="fixed">
-        <origin xyz="$(optenv CPR_LASER_XYZ 0 0 0)" rpy="$(optenv CPR_LASER_RPY 0 0 0)" />
-        <parent link="$(optenv CPR_LASER_PARENT base_link)" />
-        <child link="$(optenv CPR_LASER_PARENT base_link)_laser" />
-      </joint>
     </xacro:if>
     <xacro:if value="${lidar_model == 'ust10'}">
       <xacro:include filename="$(find generic_robot)/urdf/accessories/lasers/hokuyo_ust10.urdf.xacro" />
       <xacro:hokuyo_ust10 frame="$(optenv CPR_LASER_PARENT base_link)_laser" topic="$(optenv CPR_LASER_TOPIC scan)"/>
-      <joint name="$(optenv CPR_LASER_PARENT base_link)_laser_joint" type="fixed">
-        <origin xyz="$(optenv CPR_LASER_XYZ 0 0 0)" rpy="$(optenv CPR_LASER_RPY 0 0 0)" />
-        <parent link="$(optenv CPR_LASER_PARENT base_link)" />
-        <child link="$(optenv CPR_LASER_PARENT base_link)_laser" />
-      </joint>
     </xacro:if>
+    <joint name="$(optenv CPR_LASER_PARENT base_link)_laser_joint" type="fixed">
+      <origin xyz="$(optenv CPR_LASER_XYZ 0 0 0)" rpy="$(optenv CPR_LASER_RPY 0 0 0)" />
+      <parent link="$(optenv CPR_LASER_PARENT base_link)" />
+      <child link="$(optenv CPR_LASER_PARENT base_link)_laser" />
+    </joint>
   </xacro:if>
   <!--
-    Add/remove a 3D lidar sensor by changing the CPR_LASER_3D environment variable. The default lidar model is the Velodyne VLP16, but this can be changed with the CPR_LASER_3D_MODEL environment variable. Valid model designations are:
+    Add/remove a 3D lidar sensor by changing the CPR_LASER_3D environment variable. The default model is the Velodyne VLP16, but this can be changed with the CPR_LASER_3D_MODEL environment variable. Valid model designations are:
     - vlp16 (default)  :: Velodyne VLP16
     - vlp32e           :: Velodyne HDL-32E
@@ -50,4 +45,25 @@
   </xacro:if>
   <!--
+    Add/remove a GNSS/GPS sensor by changing the CPR_NAVSAT environment variable. The default model is the Novatel SMART7, but this can be changed with the CPR_NAVSAT_MODEL environment variable. Valid model designations are:
+    - smart7 (default)  :: Novatel SMART7
+    - smart6            :: Novatel SMART6
+  -->
+  <xacro:if value="$(optenv CPR_NAVSAT 0)">
+    <xacro:property name="navsat_model" value="$(optenv CPR_NAVSAT_MODEL smart7)" />
+    <xacro:if value="${navsat_model == 'smart7'}">
+      <xacro:include filename="$(find generic_robot)/urdf/accessories/gps/novatel_smart7.urdf.xacro" />
+      <xacro:novatel_smart7 parent="$(optenv CPR_NAVSAT_PARENT base_link)"/>
+    </xacro:if>
+    <xacro:if value="${navsat_model == 'smart6'}">
+      <xacro:include filename="$(find generic_robot)/urdf/accessories/gps/novatel_smart6.urdf.xacro" />
+      <xacro:novatel_smart6 parent="$(optenv CPR_NAVSAT_PARENT base_link)"/>
+    </xacro:if>
+    <joint name="$(optenv CPR_NAVSAT_PARENT base_link)_navsat_joint" type="fixed">
+      <origin xyz="$(optenv CPR_NAVSAT_XYZ 0 0 0)" rpy="$(optenv CPR_NAVSAT_RPY 0 0 0)" />
+      <parent link="$(optenv CPR_NAVSAT_PARENT base_link)" />
+      <child link="$(optenv CPR_NAVSAT_PARENT base_link)_navsat" />
+    </joint>
+  </xacro:if>
+  <!--
     Add/remove a Telodyne FLIR Flea3 camera by changing the CPR_FLEA3 environment variable.
   -->

Commit message: Add GX5 IMU URDF

File: urdf/accessories.urdf.xacro (robot description, xacro)
@@ -1,4 +1,5 @@
 <?xml version="1.0"?>
 <robot xmlns:xacro="http://www.ros.org/wiki/xacro">
+  <xacro:property name="PI" value="3.1415926535897931" />
   <material name="dark_grey"><color rgba="0.2 0.2 0.2 1.0" /></material>
   <material name="black"><color rgba="0.15 0.15 0.15 1.0" /></material>
@@ -15,5 +16,5 @@
     </xacro:if>
     <xacro:if value="${lidar_model == 'ust10'}">
-      <xacro:include filename="$(find generic_robot)/urdf/accessories/lasers/hokuyo_ust10.urdf.xacro" />
+      <xacro:include filename="$(find generic_robot)/urdf/accessories/laser/hokuyo_ust10.urdf.xacro" />
       <xacro:hokuyo_ust10 frame="$(optenv CPR_LASER_PARENT base_link)_laser" topic="$(optenv CPR_LASER_TOPIC scan)"/>
     </xacro:if>
@@ -66,4 +67,21 @@
   </xacro:if>
   <!--
+    Add/remove an IMU sensor by changing the CPR_IMU environment variable. The default model is the Microstrain GX5, but this can be changed with the CPR_IMU_MODEL environment variable. Valid model designations are:
+    - gx5 (default)  :: Microstrain GX5
+  -->
+  <xacro:if value="$(optenv CPR_IMU 0)">
+    <xacro:property name="imu_model" value="$(optenv CPR_IMU_MODEL gx5)" />
+    <xacro:if value="${imu_model == 'gx5'}">
+      <xacro:include filename="$(find generic_robot)/urdf/accessories/imu/microstrain_gx5.urdf.xacro" />
+      <xacro:microstrain_gx5 parent="$(optenv CPR_IMU_PARENT base_link)"/>
+    </xacro:if>
+    <joint name="$(optenv CPR_IMU_PARENT base_link)_gx5_link_joint" type="fixed">
+      <!-- TODO This offset & rotation may not be final, but it's good enough for now.  May update, pending RSCI-10 -->
+      <origin xyz="$(optenv CPR_IMU_XYZ -0.139 0.096 0.100)" rpy="$(optenv CPR_IMU_RPY ${PI} 0 -${PI/2})" />
+      <parent link="$(optenv CPR_IMU_PARENT base_link)" />
+      <child link="$(optenv CPR_IMU_PARENT base_link)_gx5_link" />
+    </joint>
+  </xacro:if>
+  <!--
     Add/remove a Telodyne FLIR Flea3 camera by changing the CPR_FLEA3 environment variable.
   -->

Commit message: Use sick_scan instead of lms1xx

File: urdf/accessories.urdf.xacro (robot description, xacro)
@@ -12,16 +12,21 @@
     <xacro:property name="lidar_model" value="$(optenv CPR_LASER_MODEL lms1xx)" />
     <xacro:if value="${lidar_model == 'lms1xx'}">
-      <xacro:include filename="$(find lms1xx)/urdf/sick_lms1xx.urdf.xacro" />
-      <xacro:sick_lms1xx frame="$(optenv CPR_LASER_PARENT base_link)_laser" topic="$(optenv CPR_LASER_TOPIC scan)" />
+      <xacro:include filename="$(find sick_scan)/urdf/sick_lms1xx.urdf.xacro" />
+      <xacro:sick_lms_1xx name="$(optenv CPR_LASER_PARENT base_link)" ros_topic="$(optenv CPR_LASER_TOPIC scan)" />
+      <joint name="$(optenv CPR_LASER_PARENT base_link)_laser_joint" type="fixed">
+        <origin xyz="$(optenv CPR_LASER_XYZ 0 0 0)" rpy="$(optenv CPR_LASER_RPY 0 0 0)" />
+        <parent link="$(optenv CPR_LASER_PARENT base_link)" />
+        <child link="$(optenv CPR_LASER_PARENT base_link)_mount_link" />
+      </joint>
     </xacro:if>
     <xacro:if value="${lidar_model == 'ust10'}">
       <xacro:include filename="$(find generic_robot)/urdf/accessories/laser/hokuyo_ust10.urdf.xacro" />
       <xacro:hokuyo_ust10 frame="$(optenv CPR_LASER_PARENT base_link)_laser" topic="$(optenv CPR_LASER_TOPIC scan)"/>
+      <joint name="$(optenv CPR_LASER_PARENT base_link)_laser_joint" type="fixed">
+        <origin xyz="$(optenv CPR_LASER_XYZ 0 0 0)" rpy="$(optenv CPR_LASER_RPY 0 0 0)" />
+        <parent link="$(optenv CPR_LASER_PARENT base_link)" />
+        <child link="$(optenv CPR_LASER_PARENT base_link)_laser" />
+      </joint>
     </xacro:if>
-    <joint name="$(optenv CPR_LASER_PARENT base_link)_laser_joint" type="fixed">
-      <origin xyz="$(optenv CPR_LASER_XYZ 0 0 0)" rpy="$(optenv CPR_LASER_RPY 0 0 0)" />
-      <parent link="$(optenv CPR_LASER_PARENT base_link)" />
-      <child link="$(optenv CPR_LASER_PARENT base_link)_laser" />
-    </joint>
   </xacro:if>
   <!--

Commit message: Update support of FLIR FLEA3 to Blackfly S

File: urdf/accessories.urdf.xacro (robot description, xacro)
@@ -84,15 +84,15 @@
   </xacro:if>
   <!--
-    Add/remove a Telodyne FLIR Flea3 camera by changing the CPR_FLEA3 environment variable.
+    Add/remove a Telodyne FLIR Blackfly S camera by changing the CPR_BLACKFLY environment variable.
   -->
-  <xacro:if value="$(optenv CPR_FLEA3 0)">
-    <xacro:include filename="$(find pointgrey_camera_description)/urdf/pointgrey_flea3.urdf.xacro" />
-    <xacro:pointgrey_flea3 frame="$(optenv CPR_FLEA3_PARENT base_link)_camera" name="$(optenv CPR_FLEA3_PARENT base_link)_camera"
+  <xacro:if value="$(optenv CPR_BLACKFLY 0)">
+    <xacro:include filename="$(find flir_camera_description)/urdf/flir_blackflys.urdf.xacro" />
+    <xacro:flir_blackflys frame="$(optenv CPR_BLACKFLY_PARENT base_link)_camera" name="$(optenv CPR_BLACKFLY_PARENT base_link)_camera"
       camera_x="0.0754" camera_y="0.029" camera_z="0.029"
       camera_mass="0.085" hfov="1.0471975512" fps="60" width="640" height="512"/>
-    <joint name="$(optenv CPR_FLEA3_PARENT base_link)_camera_joint" type="fixed">
-      <origin xyz="$(optenv CPR_FLEA3_XYZ 0 0 0)" rpy="$(optenv CPR_FLEA3_RPY 0 0 0)" />
-      <parent link="$(optenv CPR_FLEA3_PARENT base_link)" />
-      <child link="$(optenv CPR_FLEA3_PARENT base_link)_camera" />
+    <joint name="$(optenv CPR_BLACKFLY_PARENT base_link)_camera_joint" type="fixed">
+      <origin xyz="$(optenv CPR_BLACKFLY_XYZ 0 0 0)" rpy="$(optenv CPR_BLACKFLY_RPY 0 0 0)" />
+      <parent link="$(optenv CPR_BLACKFLY_PARENT base_link)" />
+      <child link="$(optenv CPR_BLACKFLY_PARENT base_link)_camera" />
     </joint>
   </xacro:if>

Commit message: Rename envars from _HOST to _IP, and from _NAVSAT to _GPS

File: urdf/accessories.urdf.xacro (robot description, xacro)
@@ -51,17 +51,17 @@
   </xacro:if>
   <!--
-    Add/remove a GNSS/GPS sensor by changing the CPR_NAVSAT environment variable. The default model is the Novatel SMART7, but this can be changed with the CPR_NAVSAT_MODEL environment variable. Valid model designations are:
+    Add/remove a GNSS/GPS sensor by changing the CPR_GPS environment variable. The default model is the Novatel SMART7, but this can be changed with the CPR_GPS_MODEL environment variable. Valid model designations are:
     - smart7 (default)  :: Novatel SMART7
   -->
-  <xacro:if value="$(optenv CPR_NAVSAT 0)">
-    <xacro:property name="navsat_model" value="$(optenv CPR_NAVSAT_MODEL smart7)" />
-    <xacro:if value="${navsat_model == 'smart7'}">
+  <xacro:if value="$(optenv CPR_GPS 0)">
+    <xacro:property name="gps_model" value="$(optenv CPR_GPS_MODEL smart7)" />
+    <xacro:if value="${gps_model == 'smart7'}">
       <xacro:include filename="$(find generic_robot)/urdf/accessories/gps/novatel_smart7.urdf.xacro" />
-      <xacro:novatel_smart7 parent="$(optenv CPR_NAVSAT_PARENT base_link)"/>
+      <xacro:novatel_smart7 parent="$(optenv CPR_GPS_PARENT base_link)"/>
     </xacro:if>
-    <joint name="$(optenv CPR_NAVSAT_PARENT base_link)_navsat_joint" type="fixed">
-      <origin xyz="$(optenv CPR_NAVSAT_XYZ 0 0 0)" rpy="$(optenv CPR_NAVSAT_RPY 0 0 0)" />
-      <parent link="$(optenv CPR_NAVSAT_PARENT base_link)" />
-      <child link="$(optenv CPR_NAVSAT_PARENT base_link)_navsat" />
+    <joint name="$(optenv CPR_GPS_PARENT base_link)_gps_joint" type="fixed">
+      <origin xyz="$(optenv CPR_GPS_XYZ 0 0 0)" rpy="$(optenv CPR_GPS_RPY 0 0 0)" />
+      <parent link="$(optenv CPR_GPS_PARENT base_link)" />
+      <child link="$(optenv CPR_GPS_PARENT base_link)_gps" />
     </joint>
   </xacro:if>

File: urdf/accessories/gps/novatel_smart6.urdf.xacro (robot description, xacro)
@@ -2,5 +2,5 @@
 <robot xmlns:xacro="http://www.ros.org/wiki/xacro">
   <xacro:macro name="novatel_smart6" params="parent">
-  <link name="${parent}_navsat">
+  <link name="${parent}_gps">
     <visual>
       <origin xyz="0 0 0" rpy="0 0 0" />

File: urdf/accessories/gps/novatel_smart7.urdf.xacro (robot description, xacro)
@@ -2,5 +2,5 @@
 <robot xmlns:xacro="http://www.ros.org/wiki/xacro">
   <xacro:macro name="novatel_smart7" params="parent">
-    <link name="${parent}_navsat">
+    <link name="${parent}_gps">
       <visual>
         <origin xyz="-0.095 0 0" rpy="${pi/2} 0 -${pi/2}" />

Commit message: Specify CPR_IMU as CPR_MICROSTRAIN for microstrain family of IMU devices; add general URDF for microstrain IMU devices

File: urdf/accessories.urdf.xacro (robot description, xacro)
@@ -67,18 +67,13 @@
   </xacro:if>
   <!--
-    Add/remove an IMU sensor by changing the CPR_IMU environment variable. The default model is the Microstrain GX5, but this can be changed with the CPR_IMU_MODEL environment variable. Valid model designations are:
-    - gx5 (default)  :: Microstrain GX5
+    Add/remove an IMU sensor by changing the CPR_MICROSTRAIN environment variable. This supports the Microstrain GX3, GX4, GX5, CX5, RQ1 and GQ7 series IMU sensors.
   -->
-  <xacro:if value="$(optenv CPR_IMU 0)">
-    <xacro:property name="imu_model" value="$(optenv CPR_IMU_MODEL gx5)" />
-    <xacro:if value="${imu_model == 'gx5'}">
-      <xacro:include filename="$(find generic_robot)/urdf/accessories/imu/microstrain_gx5.urdf.xacro" />
-      <xacro:microstrain_gx5 parent="$(optenv CPR_IMU_PARENT base_link)"/>
-    </xacro:if>
-    <joint name="$(optenv CPR_IMU_PARENT base_link)_gx5_link_joint" type="fixed">
-      <!-- TODO This offset & rotation may not be final, but it's good enough for now.  May update, pending RSCI-10 -->
-      <origin xyz="$(optenv CPR_IMU_XYZ -0.139 0.096 0.100)" rpy="$(optenv CPR_IMU_RPY ${PI} 0 -${PI/2})" />
-      <parent link="$(optenv CPR_IMU_PARENT base_link)" />
-      <child link="$(optenv CPR_IMU_PARENT base_link)_gx5_link" />
+  <xacro:if value="$(optenv CPR_MICROSTRAIN 0)">
+    <xacro:include filename="$(find generic_robot)/urdf/accessories/imu/microstrain.urdf.xacro" />
+    <xacro:microstrain />
+    <joint name="$(optenv CPR_MICROSTRAIN_PARENT base_link)_microstrain_link_joint" type="fixed">
+      <origin xyz="$(optenv CPR_MICROSTRAIN_XYZ 0 0 0)" rpy="$(optenv CPR_MICROSTRAIN_RPY 0 0 0)" />
+      <parent link="$(optenv CPR_MICROSTRAIN_PARENT base_link)" />
+      <child link="microstrain_link" />
     </joint>
   </xacro:if>

Commit message: Add Garmin GPS support; update some link names

File: urdf/accessories.urdf.xacro (robot description, xacro)
@@ -1,5 +1,4 @@
 <?xml version="1.0"?>
 <robot xmlns:xacro="http://www.ros.org/wiki/xacro">
-  <xacro:property name="PI" value="3.1415926535897931" />
   <material name="dark_grey"><color rgba="0.2 0.2 0.2 1.0" /></material>
   <material name="black"><color rgba="0.15 0.15 0.15 1.0" /></material>
@@ -7,5 +6,5 @@
     Add/remove a 2D lidar sensor by changing the CPR_LASER environment variable. The default model is the SICK LMS1xx, but this can be changed with the CPR_LASER_MODEL environment variable. Valid model designations are:
     - lms1xx (default) :: SICK LMS1xx
-    - ust10            :: Hokuyo UST-10LX
+    - ust10lx          :: Hokuyo UST-10LX
   -->
   <xacro:if value="$(optenv CPR_LASER 0)">
@@ -13,18 +12,18 @@
     <xacro:if value="${lidar_model == 'lms1xx'}">
       <xacro:include filename="$(find sick_scan)/urdf/sick_lms1xx.urdf.xacro" />
-      <xacro:sick_lms_1xx name="$(optenv CPR_LASER_PARENT base_link)" ros_topic="$(optenv CPR_LASER_TOPIC scan)" />
-      <joint name="$(optenv CPR_LASER_PARENT base_link)_laser_joint" type="fixed">
+      <xacro:sick_lms_1xx name="sick_lms1xx" ros_topic="$(optenv CPR_LASER_TOPIC scan)" />
+      <joint name="$(optenv CPR_LASER_PARENT base_link)_sick_lms1xx_laser_joint" type="fixed">
         <origin xyz="$(optenv CPR_LASER_XYZ 0 0 0)" rpy="$(optenv CPR_LASER_RPY 0 0 0)" />
         <parent link="$(optenv CPR_LASER_PARENT base_link)" />
-        <child link="$(optenv CPR_LASER_PARENT base_link)_mount_link" />
+        <child link="sick_lms1xx_mount_link" />
       </joint>
     </xacro:if>
-    <xacro:if value="${lidar_model == 'ust10'}">
-      <xacro:include filename="$(find generic_robot)/urdf/accessories/laser/hokuyo_ust10.urdf.xacro" />
-      <xacro:hokuyo_ust10 frame="$(optenv CPR_LASER_PARENT base_link)_laser" topic="$(optenv CPR_LASER_TOPIC scan)"/>
-      <joint name="$(optenv CPR_LASER_PARENT base_link)_laser_joint" type="fixed">
+    <xacro:if value="${lidar_model == 'ust10lx'}">
+      <xacro:include filename="$(find generic_robot)/urdf/accessories/laser/hokuyo_ust10lx.urdf.xacro" />
+      <xacro:hokuyo_ust10lx frame="hokuyo_ust10lx_laser" topic="$(optenv CPR_LASER_TOPIC scan)"/>
+      <joint name="hokuyo_ust10lx_laser_joint" type="fixed">
         <origin xyz="$(optenv CPR_LASER_XYZ 0 0 0)" rpy="$(optenv CPR_LASER_RPY 0 0 0)" />
         <parent link="$(optenv CPR_LASER_PARENT base_link)" />
-        <child link="$(optenv CPR_LASER_PARENT base_link)_laser" />
+        <child link="hokuyo_ust10lx_laser" />
       </joint>
     </xacro:if>
@@ -51,6 +50,8 @@
   </xacro:if>
   <!--
-    Add/remove a GNSS/GPS sensor by changing the CPR_GPS environment variable. The default model is the Novatel SMART7, but this can be changed with the CPR_GPS_MODEL environment variable. Valid model designations are:
+    Add/remove a serial GNSS/GPS sensor by changing the CPR_GPS environment variable. The default model is the Novatel SMART7, but this can be changed with the CPR_GPS_MODEL environment variable. Valid model designations are:
     - smart7 (default)  :: Novatel SMART7
+    - smart6            :: Novatel SMART6
+    - 18x               :: Garmin 18x
   -->
   <xacro:if value="$(optenv CPR_GPS 0)">
@@ -58,10 +59,14 @@
     <xacro:if value="${gps_model == 'smart7'}">
       <xacro:include filename="$(find generic_robot)/urdf/accessories/gps/novatel_smart7.urdf.xacro" />
-      <xacro:novatel_smart7 parent="$(optenv CPR_GPS_PARENT base_link)"/>
+      <xacro:novatel_smart7 />
     </xacro:if>
-    <joint name="$(optenv CPR_GPS_PARENT base_link)_gps_joint" type="fixed">
+    <xacro:if value="${gps_model == '18x'}">
+      <xacro:include filename="$(find generic_robot)/urdf/accessories/gps/garmin_18x.urdf.xacro" />
+      <xacro:garmin_18x />
+    </xacro:if>
+    <joint name="$(optenv CPR_GPS_PARENT base_link)_gps_link_joint" type="fixed">
       <origin xyz="$(optenv CPR_GPS_XYZ 0 0 0)" rpy="$(optenv CPR_GPS_RPY 0 0 0)" />
       <parent link="$(optenv CPR_GPS_PARENT base_link)" />
-      <child link="$(optenv CPR_GPS_PARENT base_link)_gps" />
+      <child link="gps_link" />
     </joint>
   </xacro:if>

File: urdf/accessories/gps/novatel_smart7.urdf.xacro (robot description, xacro)
@@ -1,6 +1,6 @@
 <?xml version="1.0"?>
 <robot xmlns:xacro="http://www.ros.org/wiki/xacro">
-  <xacro:macro name="novatel_smart7" params="parent">
-    <link name="${parent}_gps">
+  <xacro:macro name="novatel_smart7" params="">
+    <link name="gps_link">
       <visual>
         <origin xyz="-0.095 0 0" rpy="${pi/2} 0 -${pi/2}" />

File: urdf/accessories/laser/hokuyo_ust10lx.urdf.xacro (robot description, xacro)
@@ -1,5 +1,5 @@
 <?xml version="1.0"?>
 <robot xmlns:xacro="http://ros.org/wiki/xacro">
-  <xacro:macro name="hokuyo_ust10" params="frame:=laser topic:=scan sample_size:=720 update_rate:=50
+  <xacro:macro name="hokuyo_ust10lx" params="frame:=laser topic:=scan sample_size:=720 update_rate:=50
               min_angle:=-2.35619 max_angle:=2.35619 min_range:=0.1 max_range:=30.0 robot_namespace:=/">
     <link name="${frame}">
@@ -8,8 +8,15 @@
         <geometry>
           <!-- Origin of this mesh is the base of the bracket. -->
-          <mesh filename="package://generic_robot/meshes/hokuyo_ust10.stl" />
+          <mesh filename="package://generic_robot/meshes/hokuyo_ust10lx.stl" />
         </geometry>
         <material name="dark_grey" />
       </visual>
+      <collision>
+        <origin xyz="0 0 0" rpy="0 0 0" />
+        <geometry>
+          <!-- Origin of this mesh is the base of the bracket. -->
+          <mesh filename="package://generic_robot/meshes/hokuyo_ust10lx.stl" />
+        </geometry>
+      </collision>
       <inertial>
         <mass value="1.1" />
