Commit message: Remove UST10 URDF; use urg_node UST10 URDF instead

File: urdf/accessories.urdf.xacro (robot description, xacro)
@@ -6,5 +6,5 @@
     Add/remove a 2D lidar sensor by changing the CPR_LASER environment variable. The default model is the SICK LMS1xx, but this can be changed with the CPR_LASER_MODEL environment variable. Valid model designations are:
     - lms1xx (default) :: SICK LMS1xx
-    - ust10lx          :: Hokuyo UST-10LX
+    - ust10            :: Hokuyo UST-10LX
   -->
   <xacro:if value="$(optenv CPR_LASER 0)">
@@ -19,12 +19,9 @@
       </joint>
     </xacro:if>
-    <xacro:if value="${lidar_model == 'ust10lx'}">
-      <xacro:include filename="$(find generic_robot)/urdf/accessories/laser/hokuyo_ust10lx.urdf.xacro" />
-      <xacro:hokuyo_ust10lx frame="hokuyo_ust10lx_laser" topic="$(optenv CPR_LASER_TOPIC scan)"/>
-      <joint name="hokuyo_ust10lx_laser_joint" type="fixed">
+    <xacro:if value="${lidar_model == 'ust10'}">
+      <xacro:include filename="$(find urg_node)/urdf/hokuyo_ust10.urdf.xacro" />
+      <xacro:hokuyo_ust10_mount topic="$(optenv CPR_LASER_TOPIC scan)" prefix="hokuyo" parent_link="$(optenv CPR_LASER_PARENT base_link)">
         <origin xyz="$(optenv CPR_LASER_XYZ 0 0 0)" rpy="$(optenv CPR_LASER_RPY 0 0 0)" />
-        <parent link="$(optenv CPR_LASER_PARENT base_link)" />
-        <child link="hokuyo_ust10lx_laser" />
-      </joint>
+      </xacro:hokuyo_ust10_mount>
     </xacro:if>
   </xacro:if>

Commit message: Remove FLIR camera support for now since it requires external SDK for driver to work

File: urdf/accessories.urdf.xacro (robot description, xacro)
@@ -80,18 +80,4 @@
   </xacro:if>
   <!--
-    Add/remove a Telodyne FLIR Blackfly S camera by changing the CPR_BLACKFLY environment variable.
-  -->
-  <xacro:if value="$(optenv CPR_BLACKFLY 0)">
-    <xacro:include filename="$(find flir_camera_description)/urdf/flir_blackflys.urdf.xacro" />
-    <xacro:flir_blackflys frame="$(optenv CPR_BLACKFLY_PARENT base_link)_camera" name="$(optenv CPR_BLACKFLY_PARENT base_link)_camera"
-      camera_x="0.0754" camera_y="0.029" camera_z="0.029"
-      camera_mass="0.085" hfov="1.0471975512" fps="60" width="640" height="512"/>
-    <joint name="$(optenv CPR_BLACKFLY_PARENT base_link)_camera_joint" type="fixed">
-      <origin xyz="$(optenv CPR_BLACKFLY_XYZ 0 0 0)" rpy="$(optenv CPR_BLACKFLY_RPY 0 0 0)" />
-      <parent link="$(optenv CPR_BLACKFLY_PARENT base_link)" />
-      <child link="$(optenv CPR_BLACKFLY_PARENT base_link)_camera" />
-    </joint>
-  </xacro:if>
-  <!--
     Add/remove an Intel RealSense family camera by changing the CPR_REALSENSE environment variable. The default model is the D435, but can be changed with the
     CPR_REALSENSE_MODEL environment variable. Valid model designations are:
