Commit message: Add Gazebo support for generic robot example

File: example/generic_robot.urdf.xacro (robot description, xacro)
@@ -56,4 +56,24 @@
       <origin xyz="${baselen*reflect/3} 0 -${wheeldiam/2+.05}" rpy="0 0 0"/>
     </joint>
+    <!-- This block provides the simulator (Gazebo) with information on a few additional
+    physical properties. See http://gazebosim.org/tutorials/?tut=ros_urdf for more-->
+    <gazebo reference="${prefix}_${suffix}_wheel">
+      <mu1 value="200.0"/>
+      <mu2 value="100.0"/>
+      <kp value="10000000.0" />
+      <kd value="1.0" />
+      <material>Gazebo/Grey</material>
+    </gazebo>
+    <!-- This block connects the wheel joint to an actuator (motor), which informs both
+    simulation and visualization of the robot -->
+    <transmission name="${prefix}_${suffix}_wheel_trans">
+      <type>transmission_interface/SimpleTransmission</type>
+      <actuator name="${prefix}_${suffix}_wheel_motor">
+        <mechanicalReduction>1</mechanicalReduction>
+      </actuator>
+      <joint name="${prefix}_${suffix}_wheel_joint">
+        <hardwareInterface>VelocityJointInterface</hardwareInterface>
+      </joint>
+    </transmission>
   </xacro:macro>
   <xacro:macro name="leg" params="prefix reflect">
@@ -117,5 +137,5 @@
     <xacro:default_inertial mass="2"/>
   </link>
-  <joint name="head_swivel" type="continuous">
+  <joint name="head_swivel" type="fixed">
     <parent link="base_link"/>
     <child link="head"/>
@@ -143,4 +163,10 @@
     <origin xyz="${.707*width+0.04} 0 ${.707*width}"/>
   </joint>
+  <!-- Gazebo plugin for ROS Control -->
+  <gazebo>
+    <plugin name="gazebo_ros_control" filename="libgazebo_ros_control.so">
+      <robotNamespace>/</robotNamespace>
+    </plugin>
+  </gazebo>
   <xacro:include filename="$(find generic_robot)/urdf/accessories.urdf.xacro" />
 </robot>

Commit message: Remove ros controllers from Gazebo for simplicity; currently out of scope

File: example/generic_robot.urdf.xacro (robot description, xacro)
@@ -56,24 +56,4 @@
       <origin xyz="${baselen*reflect/3} 0 -${wheeldiam/2+.05}" rpy="0 0 0"/>
     </joint>
-    <!-- This block provides the simulator (Gazebo) with information on a few additional
-    physical properties. See http://gazebosim.org/tutorials/?tut=ros_urdf for more-->
-    <gazebo reference="${prefix}_${suffix}_wheel">
-      <mu1 value="200.0"/>
-      <mu2 value="100.0"/>
-      <kp value="10000000.0" />
-      <kd value="1.0" />
-      <material>Gazebo/Grey</material>
-    </gazebo>
-    <!-- This block connects the wheel joint to an actuator (motor), which informs both
-    simulation and visualization of the robot -->
-    <transmission name="${prefix}_${suffix}_wheel_trans">
-      <type>transmission_interface/SimpleTransmission</type>
-      <actuator name="${prefix}_${suffix}_wheel_motor">
-        <mechanicalReduction>1</mechanicalReduction>
-      </actuator>
-      <joint name="${prefix}_${suffix}_wheel_joint">
-        <hardwareInterface>VelocityJointInterface</hardwareInterface>
-      </joint>
-    </transmission>
   </xacro:macro>
   <xacro:macro name="leg" params="prefix reflect">

Commit message: Rename package to cpr_robot_customizer; separate Gazebo and Rviz launch files

File: example/generic_robot.urdf.xacro (robot description, xacro)
@@ -150,4 +150,4 @@
   </gazebo>
   <!-- Add this line to include sensor URDFs -->
-  <xacro:include filename="$(find generic_robot)/urdf/accessories.urdf.xacro" />
+  <xacro:include filename="$(find cpr_robot_customizer)/urdf/accessories.urdf.xacro" />
 </robot>

File: urdf/accessories.urdf.xacro (robot description, xacro)
@@ -54,9 +54,9 @@
     <xacro:property name="gps_model" value="$(optenv CPR_GPS_MODEL smart7)" />
     <xacro:if value="${gps_model == 'smart7'}">
-      <xacro:include filename="$(find generic_robot)/urdf/accessories/gps/novatel_smart7.urdf.xacro" />
+      <xacro:include filename="$(find cpr_robot_customizer)/urdf/accessories/gps/novatel_smart7.urdf.xacro" />
       <xacro:novatel_smart7 />
     </xacro:if>
     <xacro:if value="${gps_model == '18x'}">
-      <xacro:include filename="$(find generic_robot)/urdf/accessories/gps/garmin_18x.urdf.xacro" />
+      <xacro:include filename="$(find cpr_robot_customizer)/urdf/accessories/gps/garmin_18x.urdf.xacro" />
       <xacro:garmin_18x />
     </xacro:if>
@@ -71,5 +71,5 @@
   -->
   <xacro:if value="$(optenv CPR_MICROSTRAIN 0)">
-    <xacro:include filename="$(find generic_robot)/urdf/accessories/imu/microstrain.urdf.xacro" />
+    <xacro:include filename="$(find cpr_robot_customizer)/urdf/accessories/imu/microstrain.urdf.xacro" />
     <xacro:microstrain />
     <joint name="$(optenv CPR_MICROSTRAIN_PARENT base_link)_microstrain_link_joint" type="fixed">
@@ -89,5 +89,5 @@
   -->
   <xacro:if value="$(optenv CPR_REALSENSE 0)">
-    <xacro:include filename="$(find generic_robot)/urdf/accessories/camera/intel_realsense.urdf.xacro" />
+    <xacro:include filename="$(find cpr_robot_customizer)/urdf/accessories/camera/intel_realsense.urdf.xacro" />
     <xacro:realsense_sensor rs_model="$(optenv CPR_REALSENSE_MODEL d435)"
                             prefix="$(optenv CPR_REALSENSE_PARENT base_link)"

File: urdf/accessories/gps/novatel_smart7.urdf.xacro (robot description, xacro)
@@ -6,5 +6,5 @@
         <origin xyz="-0.095 0 0" rpy="${pi/2} 0 -${pi/2}" />
         <geometry>
-          <mesh filename="package://generic_robot/meshes/novatel-smart7.stl"/>
+          <mesh filename="package://cpr_robot_customizer/meshes/novatel-smart7.stl"/>
         </geometry>
         <material name="novatel_white">
@@ -15,5 +15,5 @@
         <origin xyz="-0.095 0 0" rpy="${pi/2} 0 -${pi/2}" />
         <geometry>
-          <mesh filename="package://generic_robot/meshes/novatel-smart7.stl"/>
+          <mesh filename="package://cpr_robot_customizer/meshes/novatel-smart7.stl"/>
         </geometry>
       </collision>
